Commit message: Add SEALP configuration management and collision environment modules

File: wrs/robot_sim/manipulators/piper/piper_description_v100_camera.urdf (robot description, URDF)
Before this commit: robot piper_camera, 10 links, 9 joints
Links:
- link arm_base: mass 10.162548567403693 -> None
Joints:
- joint joint6: limit lower=-3.14 upper=3.14 effort=100 velocity=3 -> lower=-2.094 upper=2.094 effort=100 velocity=3; origin xyz=0 0.091 0.0014165 rpy=-1.5708 -1.5708 0 -> xyz=0 0.091 0.0014165 rpy=1.5708 0.0 3.14159
